File: SofleTestBoard.kicad_sch (KiCad schematic)
At the start: 24 parts, among them SW1 SW_PUSH-MX_W_LED, SW2 SW_PUSH-MX_W_LED, SW3 SW_PUSH-MX_W_LED, SW4 SW_PUSH-MX_W_LED, SW5 SW_PUSH-MX_W_LED, SW6 SW_PUSH-MX_W_LED, SW7 SW_PUSH-MX_W_LED, SW8 SW_PUSH-MX_W_LED, SW9 SW_PUSH-MX_W_LED, U1 Pico

Commit message: Finished initial design. No DRC run yet
Parts:
- added H5: MountingHole, symbol Mechanical:MountingHole_Pad
- added H6: MountingHole, MountingHole:MountingHole_2.5mm_Pad_TopBottom, symbol Mechanical:MountingHole_Pad
- H1: symbol Mechanical:MountingHole -> Mechanical:MountingHole_Pad
- H2, H3, H4: footprint MountingHole:MountingHole_2.5mm -> (none); symbol Mechanical:MountingHole -> Mechanical:MountingHole_Pad
- JP1: value (none) -> Jumper_3_Open; footprint (none) -> Jumper:SolderJumper-3_P1.3mm_Open_RoundedPad1.0x1.5mm_NumberLabels
Connections:
- net COL0: now also U1.25 (GPIO19)
- net COL1: now also U1.22 (GPIO17)
- net COL2: now also U1.21 (GPIO16)
- net DOUT_R0: now also SW3.3 (DIN)
- net GND: now also H1.1, H2.1, H3.1, H4.1, U1.13 (GND), U1.18 (GND), U1.23 (GND), U1.28 (GND), U1.3 (GND), U1.33 (AGND), U1.38 (GND), U1.42 (GND), U1.8 (GND), H5.1, H6.1
- net ROW0: now also U1.24 (GPIO18)
- net ROW1: now also U1.26 (GPIO20)
- net ROW2: now also U1.32 (GPIO27_ADC1)
