File: SofleTestBoard.kicad_pcb (KiCad board)
At the start: 2 copper layers, 100 x 63.5 mm, 23 parts, among them SW1 SW_PUSH-MX_W_LED, SW2 SW_PUSH-MX_W_LED, SW3 SW_PUSH-MX_W_LED, SW4 SW_PUSH-MX_W_LED, SW5 SW_PUSH-MX_W_LED, SW6 SW_PUSH-MX_W_LED, SW7 SW_PUSH-MX_W_LED, SW8 SW_PUSH-MX_W_LED, SW9 SW_PUSH-MX_W_LED, U1 Pico

Commit message: Finished initial design. No DRC run yet
Parts:
- added H5: MountingHole, MountingHole:MountingHole_2.5mm_Pad_TopBottom, F.Cu at (159.0, 79.8)
- added H6: MountingHole, MountingHole:MountingHole_2.5mm_Pad_TopBottom, F.Cu at (120.0, 79.8)
- added JP1: Jumper_3_Open, Jumper:SolderJumper-3_P1.3mm_Open_RoundedPad1.0x1.5mm_NumberLabels, B.Cu at (177.0, 64.0)
- H1, H2, H3, H4: footprint MountingHole:MountingHole_2.5mm -> MountingHole:MountingHole_2.5mm_Pad_TopBottom
- moved U1 10.1 mm to (104.2, 82.6), turned to 180 degrees
- moved H3 1.50 mm to (178.0, 105.0)
- moved H4 1.50 mm to (84.0, 105.0)
Connections:
- SW3 pad 3: unconnected-(SW3-Pad3) -> /DOUT_R0
- U1 pad 13: unconnected-(U1-Pad13) -> GND
- U1 pad 18: unconnected-(U1-Pad18) -> GND
- U1 pad 21: unconnected-(U1-Pad21) -> /COL2
- U1 pad 22: unconnected-(U1-Pad22) -> /COL1
- U1 pad 23: unconnected-(U1-Pad23) -> GND
- U1 pad 24: unconnected-(U1-Pad24) -> /ROW0
- U1 pad 25: unconnected-(U1-Pad25) -> /COL0
- U1 pad 26: unconnected-(U1-Pad26) -> /ROW1
- U1 pad 28: unconnected-(U1-Pad28) -> GND
- U1 pad 3: unconnected-(U1-Pad3) -> GND
- U1 pad 32: unconnected-(U1-Pad32) -> /ROW2
- U1 pad 33: unconnected-(U1-Pad33) -> GND
- U1 pad 38: unconnected-(U1-Pad38) -> GND
- U1 pad 42: unconnected-(U1-Pad42) -> GND
- U1 pad 8: unconnected-(U1-Pad8) -> GND
Routing:
- net /COL2: track 92.8 -> 175.2 mm, vias 3 -> 4
- net /COL1: track 92.7 -> 156.3 mm, vias 3 -> 4
- net GND: track 0.00 -> 38.5 mm, vias 0 -> 80
- net /ROW0: track 60.2 -> 97.8 mm, vias 3 -> 4
- net /COL0: track 97.3 -> 129.2 mm, vias 3 -> 4
- net /ROW2: track 55.4 -> 83.9 mm, vias 3 -> 5
- net /ROW1: track 59.7 -> 87.8 mm, vias 3 -> 5
- net unconnected-(U1-Pad21): track 19.5 -> 0.00 mm, vias 1 -> 0
- net unconnected-(U1-Pad13): track 18.6 -> 0.00 mm, vias 1 -> 0
- net unconnected-(U1-Pad33): track 18.4 -> 0.00 mm, vias 1 -> 0
- net unconnected-(U1-Pad22): track 18.4 -> 0.00 mm, vias 1 -> 0
- net unconnected-(U1-Pad25): track 18.3 -> 0.00 mm, vias 1 -> 0
- net unconnected-(U1-Pad23): track 18.3 -> 0.00 mm, vias 1 -> 0
- net unconnected-(U1-Pad26): track 18.3 -> 0.00 mm, vias 1 -> 0
- net unconnected-(U1-Pad32): track 18.3 -> 0.00 mm, vias 1 -> 0
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Other:
- board size 100 x 63.5 mm -> 100 x 62 mm
- board text added: "SofleTestBoard by Freeviv"

Commit message: DRC setup and executed
Routing:
- net GND: track 38.5 -> 0.90 mm, vias 80 -> 74
- net VBUS: track 269.5 -> 273.5 mm
- net unconnected-(U1-Pad1): track 19.3 -> 22.4 mm
- net unconnected-(U1-Pad39): track 19.3 -> 21.2 mm
- net /ROW0: track 97.8 -> 96.1 mm
- net unconnected-(U1-Pad2): track 20.0 -> 21.1 mm
- net /COL0: track 129.2 -> 128.3 mm
- net /ROW2: track 83.9 -> 83.1 mm
- net /DOUT_R2: track 88.7 -> 89.3 mm
- net (no net): vias 1 -> 0
